File: minicurso/minicurso.sch (KiCad schematic (older format))
At the start: 17 parts

Commit message: Adicionar anotacoes
Parts:
- gave numbers to parts that had none: 15
- renumbered R to R2, R to R3
Changed lines of the file:
@@
 $EndDescr
 $Comp
-L MCU_Microchip_ATmega:ATmega32U4-AU U?
+L MCU_Microchip_ATmega:ATmega32U4-AU U1
 U 1 1 5D7A3DE3
 P 4000 3000
-F 0 "U?" H 4000 1850 50  0000 C CNN
+F 0 "U1" H 4000 1850 50  0000 C CNN
 F 1 "ATmega32U4-AU" H 4000 1750 50  0000 C CNN
 F 2 "Package_QFP:TQFP-44_10x10mm_P0.8mm" H 4000 3000 50  0001 C CIN
@@
 $EndComp
 $Comp
-L Connector:USB_B_Micro J?
+L Connector:USB_B_Micro J1
 U 1 1 5D7A3F22
 P 2450 2500
-F 0 "J?" H 2300 2950 50  0000 C CNN
+F 0 "J1" H 2300 2950 50  0000 C CNN
 F 1 "USB_B_Micro" H 2350 2850 50  0000 C CNN
 F 2 "" H 2600 2450 50  0001 C CNN
@@
 	3200 2600 3400 2600
 $Comp
-L Device:R R
+L Device:R R2
 U 1 1 5D7A4381
 P 3050 2500
-F 0 "R" V 2950 2500 50  0000 C CNN
+F 0 "R2" V 2950 2500 50  0000 C CNN
 F 1 "22R" V 3050 2500 50  0000 C CNN
 F 2 "" V 2980 2500 50  0001 C CNN
@@
 $EndComp
 $Comp
-L Device:R R
+L Device:R R3
 U 1 1 5D7A44B1
 P 3050 2600
-F 0 "R" V 3150 2600 50  0000 C CNN
+F 0 "R3" V 3150 2600 50  0000 C CNN
 F 1 "22R" V 3050 2600 50  0000 C CNN
 F 2 "" V 2980 2600 50  0001 C CNN
@@
 $EndComp
 $Comp
-L power:GND #PWR?
+L power:GND #PWR04
 U 1 1 5D7A4791
 P 2450 2900
-F 0 "#PWR?" H 2450 2650 50  0001 C CNN
+F 0 "#PWR04" H 2450 2650 50  0001 C CNN
 F 1 "GND" H 2455 2727 50  0000 C CNN
 F 2 "" H 2450 2900 50  0001 C CNN
@@
 $EndComp
 $Comp
-L power:GND #PWR?
+L power:GND #PWR010
 U 1 1 5D7A4F01
 P 3950 4850
-F 0 "#PWR?" H 3950 4600 50  0001 C CNN
+F 0 "#PWR010" H 3950 4600 50  0001 C CNN
 F 1 "GND" H 3955 4677 50  0000 C CNN
 F 2 "" H 3950 4850 50  0001 C CNN
@@
 	4000 4850 4000 4800
 $Comp
-L Device:Crystal Y?
+L Device:Crystal Y1
 U 1 1 5D7A53EA
 P 3200 1800
-F 0 "Y?" V 3100 1550 50  0000 L CNN
+F 0 "Y1" V 3100 1550 50  0000 L CNN
 F 1 "16MHz" V 3200 1400 50  0000 L CNN
 F 2 "" H 3200 1800 50  0001 C CNN
@@
 	3200 1650 3400 1650
 $Comp
-L Device:C C?
+L Device:C C2
 U 1 1 5D7A6541
 P 3200 1500
-F 0 "C?" H 2950 1600 50  0000 L CNN
+F 0 "C2" H 2950 1600 50  0000 L CNN
 F 1 "15pF" H 2900 1500 50  0000 L CNN
 F 2 "" H 3238 1350 50  0001 C CNN
@@
 Connection ~ 3200 1650
 $Comp
-L power:GND #PWR?
+L power:GND #PWR06
 U 1 1 5D7A65E6
 P 3200 1350
-F 0 "#PWR?" H 3200 1100 50  0001 C CNN
+F 0 "#PWR06" H 3200 1100 50  0001 C CNN
 F 1 "GND" H 3200 1200 50  0000 C CNN
 F 2 "" H 3200 1350 50  0001 C CNN
@@
 $EndComp
 $Comp
-L Device:C C?
+L Device:C C3
 U 1 1 5D7A66D4
 P 3200 2100
-F 0 "C?" H 2950 2200 50  0000 L CNN
+F 0 "C3" H 2950 2200 50  0000 L CNN
 F 1 "15pF" H 2900 2100 50  0000 L CNN
 F 2 "" H 3238 1950 50  0001 C CNN
@@
 Connection ~ 3200 1950
 $Comp
-L power:GND #PWR?
+L power:GND #PWR07
 U 1 1 5D7A6801
 P 3200 2250
-F 0 "#PWR?" H 3200 2000 50  0001 C CNN
+F 0 "#PWR07" H 3200 2000 50  0001 C CNN
 F 1 "GND" H 3100 2250 50  0000 C CNN
 F 2 "" H 3200 2250 50  0001 C CNN
@@
 $EndComp
 $Comp
-L power:+5V #PWR?
+L power:+5V #PWR05
 U 1 1 5D7A6D12
 P 2750 2300
-F 0 "#PWR?" H 2750 2150 50  0001 C CNN
+F 0 "#PWR05" H 2750 2150 50  0001 C CNN
 F 1 "+5V" H 2765 2473 50  0000 C CNN
 F 2 "" H 2750 2300 50  0001 C CNN
@@
 $EndComp
 $Comp
-L power:+5V #PWR?
+L power:+5V #PWR08
 U 1 1 5D7A6EC6
 P 3400 2300
-F 0 "#PWR?" H 3400 2150 50  0001 C CNN
+F 0 "#PWR08" H 3400 2150 50  0001 C CNN
 F 1 "+5V" H 3400 2250 50  0000 C CNN
 F 2 "" H 3400 2300 50  0001 C CNN
@@
 $EndComp
 $Comp
-L Device:C C?
+L Device:C C4
 U 1 1 5D7A6F9F
 P 3400 2950
-F 0 "C?" H 3150 3050 50  0000 L CNN
+F 0 "C4" H 3150 3050 50  0000 L CNN
 F 1 "1uF" H 3150 2950 50  0000 L CNN
 F 2 "" H 3438 2800 50  0001 C CNN
@@
 $EndComp
 $Comp
-L power:GND #PWR?
+L power:GND #PWR09
 U 1 1 5D7A6FFB
 P 3400 3100
-F 0 "#PWR?" H 3400 2850 50  0001 C CNN
+F 0 "#PWR09" H 3400 2850 50  0001 C CNN
 F 1 "GND" H 3405 2927 50  0000 C CNN
 F 2 "" H 3400 3100 50  0001 C CNN
@@
 $EndComp
 $Comp
-L power:+5V #PWR?
+L power:+5V #PWR012
 U 1 1 5D7A4BAC
 P 4800 700
-F 0 "#PWR?" H 4800 550 50  0001 C CNN
+F 0 "#PWR012" H 4800 550 50  0001 C CNN
 F 1 "+5V" H 4815 873 50  0000 C CNN
 F 2 "" H 4800 700 50  0001 C CNN
@@
 $EndComp
 $Comp
-L Device:C C?
+L Device:C C5
 U 1 1 5D7A7E2D
 P 4800 850
-F 0 "C?" H 4915 896 50  0000 L CNN
+F 0 "C5" H 4915 896 50  0000 L CNN
 F 1 "1u" H 4915 805 50  0000 L CNN
 F 2 "" H 4838 700 50  0001 C CNN
@@
 $EndComp
 $Comp
-L power:GND #PWR?
+L power:GND #PWR013
 U 1 1 5D7A7F18
 P 4800 1000
-F 0 "#PWR?" H 4800 750 50  0001 C CNN
+F 0 "#PWR013" H 4800 750 50  0001 C CNN
 F 1 "GND" H 4805 827 50  0000 C CNN
 F 2 "" H 4800 1000 50  0001 C CNN
@@
 $EndComp
 $Comp
-L Device:C C?
+L Device:C C6
 U 1 1 5D7A81A9
 P 5300 850
-F 0 "C?" H 5415 896 50  0000 L CNN
+F 0 "C6" H 5415 896 50  0000 L CNN
 F 1 "100n" H 5415 805 50  0000 L CNN
 F 2 "" H 5338 700 50  0001 C CNN
@@
 $EndComp
 $Comp
-L power:+5V #PWR?
+L power:+5V #PWR014
 U 1 1 5D7A8211
 P 5300 700
-F 0 "#PWR?" H 5300 550 50  0001 C CNN
+F 0 "#PWR014" H 5300 550 50  0001 C CNN
 F 1 "+5V" H 5315 873 50  0000 C CNN
 F 2 "" H 5300 700 50  0001 C CNN
@@
 $EndComp
 $Comp
-L power:GND #PWR?
+L power:GND #PWR015
 U 1 1 5D7A8230
 P 5300 1000
-F 0 "#PWR?" H 5300 750 50  0001 C CNN
+F 0 "#PWR015" H 5300 750 50  0001 C CNN
 F 1 "GND" H 5305 827 50  0000 C CNN
 F 2 "" H 5300 1000 50  0001 C CNN
@@
 $EndComp
 $Comp
-L Device:C C?
+L Device:C C7
 U 1 1 5D7A841B
 P 5800 850
-F 0 "C?" H 5915 896 50  0000 L CNN
+F 0 "C7" H 5915 896 50  0000 L CNN
 F 1 "100n" H 5915 805 50  0000 L CNN
 F 2 "" H 5838 700 50  0001 C CNN
@@
 $EndComp
 $Comp
-L power:+5V #PWR?
+L power:+5V #PWR016
 U 1 1 5D7A8457
 P 5800 700
-F 0 "#PWR?" H 5800 550 50  0001 C CNN
+F 0 "#PWR016" H 5800 550 50  0001 C CNN
 F 1 "+5V" H 5815 873 50  0000 C CNN
 F 2 "" H 5800 700 50  0001 C CNN
@@
 $EndComp
 $Comp
-L power:GND #PWR?
+L power:GND #PWR017
 U 1 1 5D7A8478
 P 5800 1000
-F 0 "#PWR?" H 5800 750 50  0001 C CNN
+F 0 "#PWR017" H 5800 750 50  0001 C CNN
 F 1 "GND" H 5805 827 50  0000 C CNN
 F 2 "" H 5800 1000 50  0001 C CNN
@@
 $EndComp
 $Comp
-L power:+5V #PWR?
+L power:+5V #PWR011
 U 1 1 5D7A8686
 P 4000 1050
-F 0 "#PWR?" H 4000 900 50  0001 C CNN
+F 0 "#PWR011" H 4000 900 50  0001 C CNN
 F 1 "+5V" H 4015 1223 50  0000 C CNN
 F 2 "" H 4000 1050 50  0001 C CNN
@@
 	4100 1050 4000 1050
 $Comp
-L Switch:SW_Push SW?
+L Switch:SW_Push SW1
 U 1 1 5D7A8A82
 P 1550 1100
-F 0 "SW?" H 1550 1385 50  0000 C CNN
+F 0 "SW1" H 1550 1385 50  0000 C CNN
 F 1 "SW_Push" H 1550 1294 50  0000 C CNN
 F 2 "" H 1550 1300 50  0001 C CNN
@@
 $EndComp
 $Comp
-L power:GND #PWR?
+L power:GND #PWR01
 U 1 1 5D7A8C8D
 P 1350 1100
-F 0 "#PWR?" H 1350 850 50  0001 C CNN
+F 0 "#PWR01" H 1350 850 50  0001 C CNN
 F 1 "GND" H 1355 927 50  0000 C CNN
 F 2 "" H 1350 1100 50  0001 C CNN
@@
 $EndComp
 $Comp
-L Device:R R?
+L Device:R R1
 U 1 1 5D7A8D6B
 P 2150 800
-F 0 "R?" V 2050 800 50  0000 C CNN
+F 0 "R1" V 2050 800 50  0000 C CNN
 F 1 "10K" V 2150 800 50  0000 C CNN
 F 2 "" V 2080 800 50  0001 C CNN
@@
 $EndComp
 $Comp
-L power:+5V #PWR?
+L power:+5V #PWR02
 U 1 1 5D7A8DFE
 P 2000 800
-F 0 "#PWR?" H 2000 650 50  0001 C CNN
+F 0 "#PWR02" H 2000 650 50  0001 C CNN
 F 1 "+5V" H 2015 973 50  0000 C CNN
 F 2 "" H 2000 800 50  0001 C CNN
@@
 	2400 1100 1750 1100
 $Comp
-L power:GND #PWR?
+L power:GND #PWR03
 U 1 1 5D7AA47D
 P 2400 1400
-F 0 "#PWR?" H 2400 1150 50  0001 C CNN
+F 0 "#PWR03" H 2400 1150 50  0001 C CNN
 F 1 "GND" H 2405 1227 50  0000 C CNN
 F 2 "" H 2400 1400 50  0001 C CNN
@@
 $EndComp
 $Comp
-L Device:C C?
+L Device:C C1
 U 1 1 5D7AA571
 P 2400 1250
-F 0 "C?" H 2515 1296 50  0000 L CNN
+F 0 "C1" H 2515 1296 50  0000 L CNN
 F 1 "100n" H 2515 1205 50  0000 L CNN
 F 2 "" H 2438 1100 50  0001 C CNN
@@
 $EndComp
 $Comp
-L Connector_Generic:Conn_01x10 J?
+L Connector_Generic:Conn_01x10 J2
 U 1 1 5D7AB30B
 P 5100 1900
-F 0 "J?" H 5180 1892 50  0000 L CNN
+F 0 "J2" H 5180 1892 50  0000 L CNN
 F 1 "Conn_01x10" H 5180 1801 50  0000 L CNN
 F 2 "" H 5100 1900 50  0001 C CNN
@@
 $EndComp
 $Comp
-L Connector_Generic:Conn_01x06 J?
+L Connector_Generic:Conn_01x06 J4
 U 1 1 5D7AB549
 P 5200 4100
-F 0 "J?" H 5280 4092 50  0000 L CNN
+F 0 "J4" H 5280 4092 50  0000 L CNN
 F 1 "Conn_01x06" H 5280 4001 50  0000 L CNN
 F 2 "" H 5200 4100 50  0001 C CNN
@@
 $EndComp
 $Comp
-L Connector_Generic:Conn_01x10 J?
+L Connector_Generic:Conn_01x10 J3
 U 1 1 5D7AB63B
 P 5100 3100
-F 0 "J?" H 5180 3092 50  0000 L CNN
+F 0 "J3" H 5180 3092 50  0000 L CNN
 F 1 "Conn_01x10" H 5180 3001 50  0000 L CNN
 F 2 "" H 5100 3100 50  0001 C CNN

Commit message: Adicionada as foodprints
Parts:
- removed J1: USB_B_Micro, symbol Connector:USB_B_Micro
- added J1: USB_B_Mini, Connector_USB:USB_Mini-B_AdamTech_MUSB-B5-S-VT-TSMT-1_SMD_Vertical, symbol Connector:USB_B_Mini
- C1, C2, C3, C4, C5, C6, C7: footprint (none) -> Capacitor_SMD:C_0805_2012Metric_Pad1.15x1.40mm_HandSolder
- J2, J3: footprint (none) -> Connector_PinHeader_2.54mm:PinHeader_1x10_P2.54mm_Vertical
- J4: footprint (none) -> Connector_PinHeader_2.54mm:PinHeader_1x06_P2.54mm_Vertical
- R1, R2, R3: footprint (none) -> Resistor_SMD:R_1206_3216Metric_Pad1.42x1.75mm_HandSolder
- SW1: footprint (none) -> Button_Switch_THT:SW_PUSH_6mm
- Y1: footprint (none) -> Crystal:Crystal_SMD_5032-2Pin_5.0x3.2mm_HandSoldering
Connections:
- net +5V: now also J1.1 (VBUS)
- net GND: now also J1.5 (GND)
- net at R3.2: now also J1.2 (D-)
- net at R2.2: now also J1.3 (D+)
Changed lines of the file:
@@
 encoding utf-8
 Sheet 1 1
-Title ""
-Date ""
-Rev ""
+Title "Minicurso SECOMP"
+Date "2019-09-12"
+Rev "V1"
 Comp ""
 Comment1 ""
@@
 	1    0    0    -1
 $EndComp
-$Comp
-L Connector:USB_B_Micro J1
-U 1 1 5D7A3F22
-P 2450 2500
-F 0 "J1" H 2300 2950 50  0000 C CNN
-F 1 "USB_B_Micro" H 2350 2850 50  0000 C CNN
-F 2 "" H 2600 2450 50  0001 C CNN
-F 3 "~" H 2600 2450 50  0001 C CNN
-	1    2450 2500
-	1    0    0    -1
-$EndComp
 Wire Wire Line
 	2750 2500 2900 2500
@@
 F 0 "R2" V 2950 2500 50  0000 C CNN
 F 1 "22R" V 3050 2500 50  0000 C CNN
-F 2 "" V 2980 2500 50  0001 C CNN
+F 2 "Resistor_SMD:R_1206_3216Metric_Pad1.42x1.75mm_HandSolder" V 2980 2500 50  0001 C CNN
 F 3 "~" H 3050 2500 50  0001 C CNN
 	1    3050 2500
@@
 F 0 "R3" V 3150 2600 50  0000 C CNN
 F 1 "22R" V 3050 2600 50  0000 C CNN
-F 2 "" V 2980 2600 50  0001 C CNN
+F 2 "Resistor_SMD:R_1206_3216Metric_Pad1.42x1.75mm_HandSolder" V 2980 2600 50  0001 C CNN
 F 3 "~" H 3050 2600 50  0001 C CNN
 	1    3050 2600
@@
 Wire Wire Line
 	4000 4850 4000 4800
-$Comp
-L Device:Crystal Y1
-U 1 1 5D7A53EA
-P 3200 1800
-F 0 "Y1" V 3100 1550 50  0000 L CNN
-F 1 "16MHz" V 3200 1400 50  0000 L CNN
-F 2 "" H 3200 1800 50  0001 C CNN
-F 3 "~" H 3200 1800 50  0001 C CNN
-	1    3200 1800
-	0    1    1    0
-$EndComp
 Wire Wire Line
 	3400 1650 3400 1700
@@
 F 0 "C2" H 2950 1600 50  0000 L CNN
 F 1 "15pF" H 2900 1500 50  0000 L CNN
-F 2 "" H 3238 1350 50  0001 C CNN
+F 2 "Capacitor_SMD:C_0805_2012Metric_Pad1.15x1.40mm_HandSolder" H 3238 1350 50  0001 C CNN
 F 3 "~" H 3200 1500 50  0001 C CNN
 	1    3200 1500
 	1    0    0    -1
 $EndComp
-Connection ~ 3200 1650
 $Comp
 L power:GND #PWR06
@@
 F 0 "C3" H 2950 2200 50  0000 L CNN
 F 1 "15pF" H 2900 2100 50  0000 L CNN
-F 2 "" H 3238 1950 50  0001 C CNN
+F 2 "Capacitor_SMD:C_0805_2012Metric_Pad1.15x1.40mm_HandSolder" H 3238 1950 50  0001 C CNN
 F 3 "~" H 3200 2100 50  0001 C CNN
 	1    3200 2100
 	1    0    0    -1
 $EndComp
-Connection ~ 3200 1950
 $Comp
 L power:GND #PWR07
@@
 F 0 "C4" H 3150 3050 50  0000 L CNN
 F 1 "1uF" H 3150 2950 50  0000 L CNN
-F 2 "" H 3438 2800 50  0001 C CNN
+F 2 "Capacitor_SMD:C_0805_2012Metric_Pad1.15x1.40mm_HandSolder" H 3438 2800 50  0001 C CNN
 F 3 "~" H 3400 2950 50  0001 C CNN
 	1    3400 2950
@@
 F 0 "C5" H 4915 896 50  0000 L CNN
 F 1 "1u" H 4915 805 50  0000 L CNN
-F 2 "" H 4838 700 50  0001 C CNN
+F 2 "Capacitor_SMD:C_0805_2012Metric_Pad1.15x1.40mm_HandSolder" H 4838 700 50  0001 C CNN
 F 3 "~" H 4800 850 50  0001 C CNN
 	1    4800 850
@@
 F 0 "C6" H 5415 896 50  0000 L CNN
 F 1 "100n" H 5415 805 50  0000 L CNN
-F 2 "" H 5338 700 50  0001 C CNN
+F 2 "Capacitor_SMD:C_0805_2012Metric_Pad1.15x1.40mm_HandSolder" H 5338 700 50  0001 C CNN
 F 3 "~" H 5300 850 50  0001 C CNN
 	1    5300 850
@@
 F 0 "C7" H 5915 896 50  0000 L CNN
 F 1 "100n" H 5915 805 50  0000 L CNN
-F 2 "" H 5838 700 50  0001 C CNN
+F 2 "Capacitor_SMD:C_0805_2012Metric_Pad1.15x1.40mm_HandSolder" H 5838 700 50  0001 C CNN
 F 3 "~" H 5800 850 50  0001 C CNN
 	1    5800 850
@@
 F 0 "SW1" H 1550 1385 50  0000 C CNN
 F 1 "SW_Push" H 1550 1294 50  0000 C CNN
-F 2 "" H 1550 1300 50  0001 C CNN
+F 2 "Button_Switch_THT:SW_PUSH_6mm" H 1550 1300 50  0001 C CNN
 F 3 "" H 1550 1300 50  0001 C CNN
 	1    1550 1100
@@
 F 0 "R1" V 2050 800 50  0000 C CNN
 F 1 "10K" V 2150 800 50  0000 C CNN
-F 2 "" V 2080 800 50  0001 C CNN
+F 2 "Resistor_SMD:R_1206_3216Metric_Pad1.42x1.75mm_HandSolder" V 2080 800 50  0001 C CNN
 F 3 "~" H 2150 800 50  0001 C CNN
 	1    2150 800
@@
 F 0 "C1" H 2515 1296 50  0000 L CNN
 F 1 "100n" H 2515 1205 50  0000 L CNN
-F 2 "" H 2438 1100 50  0001 C CNN
+F 2 "Capacitor_SMD:C_0805_2012Metric_Pad1.15x1.40mm_HandSolder" H 2438 1100 50  0001 C CNN
 F 3 "~" H 2400 1250 50  0001 C CNN
 	1    2400 1250
@@
 F 0 "J2" H 5180 1892 50  0000 L CNN
 F 1 "Conn_01x10" H 5180 1801 50  0000 L CNN
-F 2 "" H 5100 1900 50  0001 C CNN
+F 2 "Connector_PinHeader_2.54mm:PinHeader_1x10_P2.54mm_Vertical" H 5100 1900 50  0001 C CNN
 F 3 "~" H 5100 1900 50  0001 C CNN
 	1    5100 1900
@@
 F 0 "J4" H 5280 4092 50  0000 L CNN
 F 1 "Conn_01x06" H 5280 4001 50  0000 L CNN
-F 2 "" H 5200 4100 50  0001 C CNN
+F 2 "Connector_PinHeader_2.54mm:PinHeader_1x06_P2.54mm_Vertical" H 5200 4100 50  0001 C CNN
 F 3 "~" H 5200 4100 50  0001 C CNN
 	1    5200 4100
@@
 F 0 "J3" H 5180 3092 50  0000 L CNN
 F 1 "Conn_01x10" H 5180 3001 50  0000 L CNN
-F 2 "" H 5100 3100 50  0001 C CNN
+F 2 "Connector_PinHeader_2.54mm:PinHeader_1x10_P2.54mm_Vertical" H 5100 3100 50  0001 C CNN
 F 3 "~" H 5100 3100 50  0001 C CNN
 	1    5100 3100
@@
 Wire Wire Line
 	4600 4400 5000 4400
+Connection ~ 3200 1950
+Connection ~ 3200 1650
+$Comp
+L Device:Crystal Y1
+U 1 1 5D7A53EA
+P 3200 1800
+F 0 "Y1" V 3100 1550 50  0000 L CNN
+F 1 "16MHz" V 3200 1400 50  0000 L CNN
+F 2 "Crystal:Crystal_SMD_5032-2Pin_5.0x3.2mm_HandSoldering" H 3200 1800 50  0001 C CNN
+F 3 "~" H 3200 1800 50  0001 C CNN
+	1    3200 1800
+	0    1    1    0
+$EndComp
+$Comp
+L Connector:USB_B_Mini J1
+U 1 1 5D7BC2A0
+P 2450 2500
+F 0 "J1" H 2505 2967 50  0000 C CNN
+F 1 "USB_B_Mini" H 2505 2876 50  0000 C CNN
+F 2 "Connector_USB:USB_Mini-B_AdamTech_MUSB-B5-S-VT-TSMT-1_SMD_Vertical" H 2600 2450 50  0001 C CNN
+F 3 "~" H 2600 2450 50  0001 C CNN
+	1    2450 2500
+	1    0    0    -1
+$EndComp
 $EndSCHEMATC
